File: breadboard_power_supply.kicad_sch (KiCad schematic)
At the start: 27 parts, among them J1 Conn_02x02_Odd_Even, J2 Conn_02x02_Odd_Even, J3 Conn_02x03_Odd_Even, J4 Conn_02x03_Odd_Even, J5 7010ASV, U1 CH224K, U2 AP63205, U3 AP2205-33Y

Commit message: part placement done, started routing of top layer
Parts:
- removed C4: 10u, 0Capacitors:C_0805_2012Metric_Pad1.18x1.45mm_HandSolder, symbol 0Capacitors:0805_10u_50v
Changed lines of the file:
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@@
-	)
-	(symbol
-		(lib_id "0Capacitors:0805_10u_50v")
-		(at 137.16 31.75 0)
-		(unit 1)
-		(exclude_from_sim no)
-		(in_bom yes)
-		(on_board yes)
-		(dnp no)
-		(property "Reference" "C4"
-			(at 137.16 29.718 0)
-			(effects
-				(font
-					(size 1.27 1.27)
-				)
-				(justify left)
-			)
-		)
-		(property "Value" "10u"
-			(at 137.16 34.036 0)
-			(effects
-				(font
-					(size 1.27 1.27)
-				)
-				(justify left)
-			)
-		)
-		(property "Footprint" "0Capacitors:C_0805_2012Metric_Pad1.18x1.45mm_HandSolder"
-			(at 136.906 40.894 0)
-			(effects
-				(font
-					(size 1.27 1.27)
-				)
-				(hide yes)
-			)
-		)
-		(property "Datasheet" ""
-			(at 137.16 31.75 0)
-			(effects
-				(font
-					(size 1.27 1.27)
-				)
-				(hide yes)
-			)
-		)
-		(property "Description" "50V 10uF X5R ±10% 0805 Multilayer Ceramic Capacitors MLCC - SMD/SMT ROHS"
-			(at 137.668 39.116 0)
-			(effects
-				(font
-					(size 1.27 1.27)
-				)
-				(hide yes)
-			)
-		)
-		(property "LCSC Part #" "C440198"
-			(at 137.16 42.672 0)
-			(effects
-				(font
-					(size 1.27 1.27)
-				)
-				(hide yes)
-			)
-		)
-		(pin "1"
-		)
-		(pin "2"
-		)
-		(instances
-			(project "breadboard_power_supply"
-				(path "/428bd1b0-cce9-4cd6-a385-fe33eda3b9ce"
-					(reference "C4")
-					(unit 1)
-				)
-			)
-		)
 	)
 	(symbol

Commit message: added production files
Parts:
- added H1, H2: MountingHole, MountingHole:MountingHole_2.2mm_M2_DIN965_Pad_TopBottom, symbol Mechanical:MountingHole
Connections:
- net VCC_PD is gone; now on net VBUS: J3.3 (Pin_3), J4.3 (Pin_3)
Changed lines of the file:
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@@
 	)
 	(symbol
+		(lib_id "Mechanical:MountingHole")
+		(at 25.4 123.19 90)
+		(unit 1)
+		(exclude_from_sim yes)
+		(in_bom no)
+		(on_board yes)
+		(dnp yes)
+		(fields_autoplaced yes)
+		(property "Reference" "H2"
+			(at 27.94 121.9199 90)
+			(effects
+				(font
+					(size 1.27 1.27)
+				)
+				(justify right)
+			)
+		)
+		(property "Value" "MountingHole"
+			(at 27.94 124.4599 90)
+			(effects
+				(font
+					(size 1.27 1.27)
+				)
+				(justify right)
+			)
+		)
+		(property "Footprint" "MountingHole:MountingHole_2.2mm_M2_DIN965_Pad_TopBottom"
+			(at 25.4 123.19 0)
+			(effects
+				(font
+					(size 1.27 1.27)
+				)
+				(hide yes)
+			)
+		)
+		(property "Datasheet" "~"
+			(at 25.4 123.19 0)
+			(effects
+				(font
+					(size 1.27 1.27)
+				)
+				(hide yes)
+			)
+		)
+		(property "Description" "Mounting Hole without connection"
+			(at 25.4 123.19 0)
+			(effects
+				(font
+					(size 1.27 1.27)
+				)
+				(hide yes)
+			)
+		)
+		(instances
+			(project "breadboard_power_supply"
+				(path "/428bd1b0-cce9-4cd6-a385-fe33eda3b9ce"
+					(reference "H2")
+					(unit 1)
+				)
+			)
+		)
+	)
+	(symbol
 		(lib_id "0Passives:0805_4.7uH_800mA")
 		(at 119.38 26.67 90)
@@
 	)
 	(symbol
+		(lib_id "Mechanical:MountingHole")
+		(at 25.4 118.11 90)
+		(unit 1)
+		(exclude_from_sim yes)
+		(in_bom no)
+		(on_board yes)
+		(dnp yes)
+		(fields_autoplaced yes)
+		(property "Reference" "H1"
+			(at 27.94 116.8399 90)
+			(effects
+				(font
+					(size 1.27 1.27)
+				)
+				(justify right)
+			)
+		)
+		(property "Value" "MountingHole"
+			(at 27.94 119.3799 90)
+			(effects
+				(font
+					(size 1.27 1.27)
+				)
+				(justify right)
+			)
+		)
+		(property "Footprint" "MountingHole:MountingHole_2.2mm_M2_DIN965_Pad_TopBottom"
+			(at 25.4 118.11 0)
+			(effects
+				(font
+					(size 1.27 1.27)
+				)
+				(hide yes)
+			)
+		)
+		(property "Datasheet" "~"
+			(at 25.4 118.11 0)
+			(effects
+				(font
+					(size 1.27 1.27)
+				)
+				(hide yes)
+			)
+		)
+		(property "Description" "Mounting Hole without connection"
+			(at 25.4 118.11 0)
+			(effects
+				(font
+					(size 1.27 1.27)
+				)
+				(hide yes)
+			)
+		)
+		(instances
+			(project ""
+				(path "/428bd1b0-cce9-4cd6-a385-fe33eda3b9ce"
+					(reference "H1")
+					(unit 1)
+				)
+			)
+		)
+	)
+	(symbol
 		(lib_id "0Capacitors:0603_100n_50v")
 		(at 82.55 107.95 0)
@@
 			)
 		)
-		(property "Value" "VCC_PD"
+		(property "Value" "VBUS"
 			(at 204.47 146.0499 90)
 			(effects
@@
 			)
 		)
-		(property "Value" "VCC_PD"
+		(property "Value" "VBUS"
 			(at 204.47 124.4599 90)
 			(effects
